File: Split_Board_PartB/MUX_OPAMP_SECTION.kicad_sch (KiCad schematic)
At the start: 158 parts, among them J1 Conn_01x28, J4 Conn_01x28, U1 MCP604, U2 MCP604

Commit message: added a BOM and a final versions of all  the files schematic and design file
Parts:
- C1: footprint Capacitor_SMD:C_0805_2012Metric_Pad1.18x1.45mm_HandSolder -> SamacSys_Parts:522072833
Changed lines of the file:
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@@
       (effects (font (size 1.27 1.27)))
     )
-    (property "Footprint" "Capacitor_SMD:C_0805_2012Metric_Pad1.18x1.45mm_HandSolder" (at 87.63 78.4098 0)
+    (property "Footprint" "SamacSys_Parts:522072833" (at 87.63 78.4098 0)
       (effects (font (size 1.27 1.27)) hide)
     )
