File: Split_Board_PartB/Split_Board_PartB.kicad_pcb (KiCad board)
At the start: 2 copper layers, 187 parts, among them IC1 CD74HC595SM96, J1 Conn_01x28, J2 Conn_01x36, J3 Conn_01x36, J4 Conn_01x28, J8 Conn_01x28, J9 Conn_01x28, U1 MCP604, U10 MCP604, U11 MCP604, U12 MCP604, U13 MCP604, U14 MCP604, U15 CD74HC4051PWT, U16 CD74HC4051PWT, U17 CD74HC4051PWT, U18 CD74HC4051PWT, U19 CD74HC4051PWT, U2 MCP604, U20 CD74HC4051PWT, U21 CD74HC4051PWT, U22 CD74HC4051PWT, U23 CD74HC4051PWT, U24 CD74HC4051PWT, U25 CD74HC4051PWT, U26 CD74HC4051PWT, U27 CD74HC4051PWT, U28 CD74HC4051PWT, U29 CD74HC4051PWT, U3 MCP604, U4 MCP604, U44 OPA187IDBVR, U5 MCP604, U6 MCP604, U7 MCP604, U8 MCP604, U9 MCP604

Commit message: added a BOM and a final versions of all  the files schematic and design file
Parts:
- removed the C28 at (127.8, 72.3)
- removed C56: 100PF, Capacitor_SMD:C_0805_2012Metric_Pad1.18x1.45mm_HandSolder
- removed the DC2 at (142.2, 72.3)
- removed IC1: CD74HC595SM96, KiCad_shift_register_cd74hc595:SOP65P780X200-16N
- removed the J2 at (89.5, 136.1)
- removed the J3 at (89.5, 147.3)
- removed the U22 at (180.4, 116.3)
- removed the U9 at (166.4, 101.6)
- added DC1: 1uf, Capacitor_SMD:C_0805_2012Metric_Pad1.18x1.45mm_HandSolder, F.Cu at (90.0, -74.6)
- added DC15: 1uf, Capacitor_SMD:C_0805_2012Metric_Pad1.18x1.45mm_HandSolder, F.Cu at (130.3, -71.7)
- added DC16: 100nf, Capacitor_SMD:C_0805_2012Metric_Pad1.18x1.45mm_HandSolder, F.Cu at (99.6, -74.6)
- added DC17: 1uf, Capacitor_SMD:C_0805_2012Metric_Pad1.18x1.45mm_HandSolder, F.Cu at (99.6, -71.6)
- added DC18: 100nf, Capacitor_SMD:C_0805_2012Metric_Pad1.18x1.45mm_HandSolder, F.Cu at (99.6, -68.6)
- added DC19: 1uf, Capacitor_SMD:C_0805_2012Metric_Pad1.18x1.45mm_HandSolder, F.Cu at (99.6, -65.6)
- added DC20: 100nf, Capacitor_SMD:C_0805_2012Metric_Pad1.18x1.45mm_HandSolder, F.Cu at (99.6, -62.6)
- added DC21: 1uf, Capacitor_SMD:C_0805_2012Metric_Pad1.18x1.45mm_HandSolder, F.Cu at (99.6, -59.6)
- added DC24: 100nf, Capacitor_SMD:C_0805_2012Metric_Pad1.18x1.45mm_HandSolder, F.Cu at (104.4, -71.6)
- added DC25: 1uf, Capacitor_SMD:C_0805_2012Metric_Pad1.18x1.45mm_HandSolder, F.Cu at (104.4, -68.6)
- added DC26: 100nf, Capacitor_SMD:C_0805_2012Metric_Pad1.18x1.45mm_HandSolder, F.Cu at (104.4, -65.6)
- added DC27: 1uf, Capacitor_SMD:C_0805_2012Metric_Pad1.18x1.45mm_HandSolder, F.Cu at (104.4, -62.6)
- added DC28: 100nf, Capacitor_SMD:C_0805_2012Metric_Pad1.18x1.45mm_HandSolder, F.Cu at (104.4, -59.6)
- added DC36: 100nF, Capacitor_SMD:C_0805_2012Metric_Pad1.18x1.45mm_HandSolder, F.Cu at (117.4, -56.6)
- added DC37: 1uF, Capacitor_SMD:C_0805_2012Metric_Pad1.18x1.45mm_HandSolder, F.Cu at (117.4, -53.6)
- added DC52: 100nF, Capacitor_SMD:C_0805_2012Metric_Pad1.18x1.45mm_HandSolder, F.Cu at (117.4, -50.6)
- added DC53: 100nF, Capacitor_SMD:C_0805_2012Metric_Pad1.18x1.45mm_HandSolder, F.Cu at (117.4, -47.6)
- added J5: Conn_01x30, Connector_FFC-FPC:Hirose_FH12-30S-0.5SH_1x30-1MP_P0.50mm_Horizontal, F.Cu at (258.6, -68.4)
- added J6: Conn_01x30, Connector_FFC-FPC:Hirose_FH12-30S-0.5SH_1x30-1MP_P0.50mm_Horizontal, F.Cu at (62.9, -67.6)
- added R57: R, Resistor_SMD:R_0805_2012Metric_Pad1.20x1.40mm_HandSolder, F.Cu at (134.7, -56.7)
- added R58: R, Resistor_SMD:R_0805_2012Metric_Pad1.20x1.40mm_HandSolder, F.Cu at (134.7, -53.7)
- added R60: 10K, Resistor_SMD:R_0805_2012Metric_Pad1.20x1.40mm_HandSolder, F.Cu at (109.2, -74.7)
- added R61: 1K, Resistor_SMD:R_0805_2012Metric_Pad1.20x1.40mm_HandSolder, F.Cu at (109.2, -71.7)
- added R62: 10K, Resistor_SMD:R_0805_2012Metric_Pad1.20x1.40mm_HandSolder, F.Cu at (109.2, -68.8)
- added R63: 1K, Resistor_SMD:R_0805_2012Metric_Pad1.20x1.40mm_HandSolder, F.Cu at (109.2, -65.8)
- added R64: 1K, Resistor_SMD:R_0805_2012Metric_Pad1.20x1.40mm_HandSolder, F.Cu at (122.2, -48.6)
- added U14: MCP604, MCP604T-I_ST:SOP65P640X120-14N, F.Cu at (119.1, -63.2)
- added U30: CD74HC595SM96, KiCad_shift_register_cd74hc595:SOP65P780X200-16N, F.Cu at (125.1, -54.1)
- added U5: MCP604, MCP604T-I_ST:SOP65P640X120-14N, F.Cu at (119.1, -75.7)
- C1: footprint Capacitor_SMD:C_0805_2012Metric_Pad1.18x1.45mm_HandSolder -> SamacSys_Parts:522072833
- DC11, DC13, DC3, DC5, DC7, DC9: value 100nf -> 1uf
- DC22: value 100nF -> 100nf
- DC23: value 100nF -> 1uf
- R55: renamed from R28; value 10K -> 0E
- R56: value 10K -> 0E
- moved DC23 209.2 mm to (104.4, -74.6)
- moved DC22 193.4 mm to (135.2, -71.7)
- moved U4 184.3 mm to (83.5, -66.8)
- moved J3 178.8 mm to (194.8, -36.9), turned to 180 degrees
- moved U2 178.6 mm to (83.5, -73.0)
- moved J2 167.8 mm to (134.1, -38.6), turned to 180 degrees
- moved J4 165.1 mm to (245.0, -36.0), turned to 180 degrees
- moved U11 162.2 mm to (119.1, -69.5)
- moved DC3 155.9 mm to (90.0, -71.6)
- moved DC4 155.9 mm to (90.0, -68.6)
- moved J1 150.9 mm to (76.7, -39.1), turned to 180 degrees
- moved R10 150.7 mm to (140.8, -72.5)
- moved R23 150.7 mm to (145.6, -75.5)
- moved R24 150.7 mm to (145.6, -72.5)
- moved R34 150.7 mm to (155.1, -75.5)
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- renumbered C25 to C17, C26 to C18, C27 to C19, C24 to C20, C17 to C21, C18 to C22, C19 to C23, C20 to C24, C21 to C25, C22 to C26, C23 to C27, C53 to C28, C54 to C29, C55 to C30, C52 to C31, C37 to C32, C38 to C33, C39 to C34, C40 to C35, C29 to C36, C30 to C37, C31 to C38, C32 to C39, C33 to C40, C34 to C41, C35 to C42, C36 to C43, C41 to C44, C42 to C45, C43 to C46, C44 to C47, C45 to C48, C46 to C49, C47 to C50, C48 to C51, C49 to C52, C50 to C53, C51 to C54, DC1 to DC2, DC15 to DC29, DC16 to DC30, DC17 to DC31, DC18 to DC32, DC19 to DC33, DC20 to DC34, DC21 to DC35, DC24 to DC38, DC25 to DC39, DC26 to DC40, DC27 to DC41, DC28 to DC42, DC29 to DC43, DC30 to DC44, DC31 to DC45, DC32 to DC46, DC33 to DC47, DC34 to DC48, DC35 to DC49, DC36 to DC50, DC37 to DC51, J4 to J1, J9 to J2, J8 to J3, J1 to J4, R25 to R17, R26 to R18, R27 to R19, R24 to R20, R17 to R21, R18 to R22, R19 to R23, R20 to R24, R21 to R25, R22 to R26, R23 to R27, R53 to R28, R54 to R29, R55 to R30, R52 to R31, R37 to R32, R38 to R33, R39 to R34, R40 to R35, R29 to R36, R30 to R37, R31 to R38, R32 to R39, R33 to R40, R34 to R41, R35 to R42, R36 to R43, R41 to R44, R42 to R45, R43 to R46, R44 to R47, R45 to R48, R46 to R49, R47 to R50, R48 to R51, R49 to R52, R50 to R53, R51 to R54, R111 to R59, U8 to U10, U5 to U12, U12 to U13, U23 to U22, U24 to U23, U25 to U24, U26 to U25, U27 to U26, U28 to U27, U29 to U28, U44 to U29, U7 to U6, U6 to U7, U14 to U8, U13 to U8, U10 to U9
Connections:
- net RS0 renamed RS0_ISO
- net RS1 renamed RS1_ISO
- net RS2 renamed RS2_ISO
- net SS0_ISO renamed CS0_ISO
- net SS1_ISO renamed CS1_ISO
- net SS2_ISO renamed CS2_ISO
- C17 pad 1: ROW_25 -> ROW_17
- C17 pad 2: M25 -> M17
- C18 pad 1: ROW_26 -> ROW_18
- C18 pad 2: M26 -> M18
- C19 pad 1: ROW_27 -> ROW_19
- C19 pad 2: M27 -> M19
- C20 pad 1: ROW_24 -> ROW_20
- C20 pad 2: M24 -> M20
- C21 pad 1: ROW_17 -> ROW_21
- C21 pad 2: M17 -> M21
- C22 pad 1: ROW_18 -> ROW_22
- C22 pad 2: M18 -> M22
- C23 pad 1: ROW_19 -> ROW_23
- C23 pad 2: M19 -> M23
- C24 pad 1: ROW_20 -> ROW_24
- C24 pad 2: M20 -> M24
- C25 pad 1: ROW_21 -> ROW_25
- C25 pad 2: M21 -> M25
- C26 pad 1: ROW_22 -> ROW_26
- C26 pad 2: M22 -> M26
- C27 pad 1: ROW_23 -> ROW_27
- C27 pad 2: M23 -> M27
- C28 pad 1: ROW_52 -> ROW_28
- C28 pad 2: M52 -> M28
- C29 pad 1: ROW_53 -> ROW_29
- C29 pad 2: M53 -> M29
- C30 pad 1: ROW_54 -> ROW_30
- C30 pad 2: M54 -> M30
- C31 pad 1: ROW_51 -> ROW_31
- C31 pad 2: M51 -> M31
- C32 pad 1: ROW_36 -> ROW_32
- C32 pad 2: M36 -> M32
- C33 pad 1: ROW_37 -> ROW_33
- C33 pad 2: M37 -> M33
- C34 pad 1: ROW_38 -> ROW_34
- C34 pad 2: M38 -> M34
- C35 pad 1: ROW_39 -> ROW_35
- C35 pad 2: M39 -> M35
- C36 pad 1: ROW_28 -> ROW_36
- C36 pad 2: M28 -> M36
- C37 pad 1: ROW_29 -> ROW_37
- C37 pad 2: M29 -> M37
- C38 pad 1: ROW_30 -> ROW_38
- C38 pad 2: M30 -> M38
- C39 pad 1: ROW_31 -> ROW_39
- C39 pad 2: M31 -> M39
- C40 pad 1: ROW_32 -> ROW_40
- C40 pad 2: M32 -> M40
- C41 pad 1: ROW_33 -> ROW_41
- C41 pad 2: M33 -> M41
- C42 pad 1: ROW_34 -> ROW_42
- C42 pad 2: M34 -> M42
- C43 pad 1: ROW_35 -> ROW_43
- C43 pad 2: M35 -> M43
- C44 pad 1: ROW_40 -> ROW_44
- C44 pad 2: M40 -> M44
- C45 pad 1: ROW_41 -> ROW_45
- C45 pad 2: M41 -> M45
- C46 pad 1: ROW_42 -> ROW_46
- C46 pad 2: M42 -> M46
- C47 pad 1: ROW_43 -> ROW_47
- C47 pad 2: M43 -> M47
- C48 pad 1: ROW_44 -> ROW_48
- C48 pad 2: M44 -> M48
- C49 pad 1: ROW_45 -> ROW_49
- C49 pad 2: M45 -> M49
- C50 pad 1: ROW_46 -> ROW_50
- C50 pad 2: M46 -> M50
- C51 pad 1: ROW_47 -> ROW_51
- C51 pad 2: M47 -> M51
- C52 pad 1: ROW_48 -> ROW_52
- C52 pad 2: M48 -> M52
- C53 pad 1: ROW_49 -> ROW_53
- C53 pad 2: M49 -> M53
- C54 pad 1: ROW_50 -> ROW_54
- C54 pad 2: M50 -> M54
- DC10 pad 1: GNDA -> GNDA_ISO
- DC11 pad 1: GNDA -> GNDA_ISO
- DC12 pad 1: GNDA -> GNDA_ISO
- DC13 pad 1: GNDA -> GNDA_ISO
- DC14 pad 1: GNDA -> GNDA_ISO
- DC2 pad 1: GNDA -> GNDA_ISO
- DC23 pad 2: -5VA_ISO -> +5VA_ISO
- DC3 pad 1: GNDA -> GNDA_ISO
- DC4 pad 1: GNDA -> GNDA_ISO
- DC5 pad 1: GNDA -> GNDA_ISO
- DC6 pad 1: GNDA -> GNDA_ISO
- DC7 pad 1: GNDA -> GNDA_ISO
- DC8 pad 1: GNDA -> GNDA_ISO
- DC9 pad 1: GNDA -> GNDA_ISO
- J1 pad 1: ROW_27 -> unconnected-(J1-Pin_1-Pad1)
- J1 pad 10: ROW_18 -> ROW_9
- J1 pad 11: ROW_17 -> ROW_10
- J1 pad 12: ROW_16 -> ROW_11
- J1 pad 13: ROW_15 -> ROW_12
- J1 pad 14: ROW_14 -> ROW_13
- J1 pad 15: ROW_13 -> ROW_14
- J1 pad 16: ROW_12 -> ROW_15
- J1 pad 17: ROW_11 -> ROW_16
- J1 pad 18: ROW_10 -> ROW_17
- J1 pad 19: ROW_9 -> ROW_18
- J1 pad 2: ROW_26 -> ROW_1
- J1 pad 20: ROW_8 -> ROW_19
- J1 pad 21: ROW_7 -> ROW_20
- J1 pad 22: ROW_6 -> ROW_21
- J1 pad 23: ROW_5 -> ROW_22
- J1 pad 24: ROW_4 -> ROW_23
- J1 pad 25: ROW_3 -> ROW_24
- J1 pad 26: ROW_2 -> ROW_25
- J1 pad 27: ROW_1 -> ROW_26
- J1 pad 28: unconnected-(J4-Pin_28-Pad28) -> ROW_27
- J1 pad 3: ROW_25 -> ROW_2
- J1 pad 4: ROW_24 -> ROW_3
- J1 pad 5: ROW_23 -> ROW_4
- J1 pad 6: ROW_22 -> ROW_5
- J1 pad 7: ROW_21 -> ROW_6
- J1 pad 8: ROW_20 -> ROW_7
- J1 pad 9: ROW_19 -> ROW_8
- J2 pad 1: COL_1 -> unconnected-(J2-Pin_1-Pad1)
- J2 pad 10: COL_10 -> COL_19
- J2 pad 11: COL_11 -> COL_18
- J2 pad 12: COL_12 -> COL_17
- J2 pad 13: COL_13 -> COL_16
- J2 pad 14: COL_14 -> COL_15
- J2 pad 15: COL_15 -> COL_14
- J2 pad 16: COL_16 -> COL_13
- J2 pad 17: COL_17 -> COL_12
- J2 pad 18: COL_18 -> COL_11
- J2 pad 19: COL_19 -> COL_10
- J2 pad 2: COL_2 -> COL_27
- J2 pad 20: COL_20 -> COL_9
- J2 pad 21: COL_21 -> COL_8
- J2 pad 22: COL_22 -> COL_7
- J2 pad 23: COL_23 -> COL_6
- J2 pad 24: COL_24 -> COL_5
- J2 pad 25: COL_25 -> COL_4
- J2 pad 26: COL_26 -> COL_3
- J2 pad 27: COL_27 -> COL_2
- J2 pad 28: unconnected-(J9-Pin_28-Pad28) -> COL_1
- J2 pad 3: COL_3 -> COL_26
- J2 pad 4: COL_4 -> COL_25
- J2 pad 5: COL_5 -> COL_24
- J2 pad 6: COL_6 -> COL_23
- J2 pad 7: COL_7 -> COL_22
- J2 pad 8: COL_8 -> COL_21
- J2 pad 9: COL_9 -> COL_20
- J3 pad 1: COL_28 -> unconnected-(J3-Pin_1-Pad1)
- J3 pad 10: COL_37 -> COL_46
- J3 pad 11: COL_38 -> COL_45
- J3 pad 12: COL_39 -> COL_44
- J3 pad 13: COL_40 -> COL_43
- J3 pad 14: COL_41 -> COL_42
- J3 pad 15: COL_42 -> COL_41
- J3 pad 16: COL_43 -> COL_40
- J3 pad 17: COL_44 -> COL_39
- J3 pad 18: COL_45 -> COL_38
- J3 pad 19: COL_46 -> COL_37
- J3 pad 2: COL_29 -> COL_54
- J3 pad 20: COL_47 -> COL_36
- J3 pad 21: COL_48 -> COL_35
- J3 pad 22: COL_49 -> COL_34
- J3 pad 23: COL_50 -> COL_33
- J3 pad 24: COL_51 -> COL_32
- J3 pad 25: COL_52 -> COL_31
- J3 pad 26: COL_53 -> COL_30
- J3 pad 27: COL_54 -> COL_29
- J3 pad 28: unconnected-(J8-Pin_28-Pad28) -> COL_28
- J3 pad 3: COL_30 -> COL_53
- J3 pad 4: COL_31 -> COL_52
- J3 pad 5: COL_32 -> COL_51
- J3 pad 6: COL_33 -> COL_50
- J3 pad 7: COL_34 -> COL_49
- J3 pad 8: COL_35 -> COL_48
- J3 pad 9: COL_36 -> COL_47
- J4 pad 1: ROW_28 -> unconnected-(J4-Pin_1-Pad1)
- J4 pad 10: ROW_37 -> ROW_46
- J4 pad 11: ROW_38 -> ROW_45
- J4 pad 12: ROW_39 -> ROW_44
- J4 pad 13: ROW_40 -> ROW_43
- J4 pad 14: ROW_41 -> ROW_42
- J4 pad 15: ROW_42 -> ROW_41
- J4 pad 16: ROW_43 -> ROW_40
- J4 pad 17: ROW_44 -> ROW_39
- J4 pad 18: ROW_45 -> ROW_38
- J4 pad 19: ROW_46 -> ROW_37
- J4 pad 2: ROW_29 -> ROW_54
- J4 pad 20: ROW_47 -> ROW_36
- J4 pad 21: ROW_48 -> ROW_35
- J4 pad 22: ROW_49 -> ROW_34
- J4 pad 23: ROW_50 -> ROW_33
- J4 pad 24: ROW_51 -> ROW_32
- J4 pad 25: ROW_52 -> ROW_31
- J4 pad 26: ROW_53 -> ROW_30
- J4 pad 27: ROW_54 -> ROW_29
- J4 pad 28: unconnected-(J1-Pin_28-Pad28) -> ROW_28
- J4 pad 3: ROW_30 -> ROW_53
- J4 pad 4: ROW_31 -> ROW_52
- J4 pad 5: ROW_32 -> ROW_51
- J4 pad 6: ROW_33 -> ROW_50
- J4 pad 7: ROW_34 -> ROW_49
- J4 pad 8: ROW_35 -> ROW_48
- J4 pad 9: ROW_36 -> ROW_47
- R17 pad 1: ROW_25 -> ROW_17
- R17 pad 2: M25 -> M17
- R18 pad 1: ROW_26 -> ROW_18
- R18 pad 2: M26 -> M18
- R19 pad 1: ROW_27 -> ROW_19
- R19 pad 2: M27 -> M19
- R20 pad 1: ROW_24 -> ROW_20
- R20 pad 2: M24 -> M20
- R21 pad 1: ROW_17 -> ROW_21
- R21 pad 2: M17 -> M21
- R22 pad 1: ROW_18 -> ROW_22
- R22 pad 2: M18 -> M22
- R23 pad 1: ROW_19 -> ROW_23
- R23 pad 2: M19 -> M23
- R24 pad 1: ROW_20 -> ROW_24
- R24 pad 2: M20 -> M24
- R25 pad 1: ROW_21 -> ROW_25
- R25 pad 2: M21 -> M25
- R26 pad 1: ROW_22 -> ROW_26
- R26 pad 2: M22 -> M26
- R27 pad 1: ROW_23 -> ROW_27
- R27 pad 2: M23 -> M27
- R28 pad 1: ROW_52 -> ROW_28
- R28 pad 2: M52 -> M28
- R29 pad 1: ROW_53 -> ROW_29
- R29 pad 2: M53 -> M29
- R30 pad 1: ROW_54 -> ROW_30
- R30 pad 2: M54 -> M30
- R31 pad 1: ROW_51 -> ROW_31
- R31 pad 2: M51 -> M31
- R32 pad 1: ROW_36 -> ROW_32
- R32 pad 2: M36 -> M32
- R33 pad 1: ROW_37 -> ROW_33
- R33 pad 2: M37 -> M33
- R34 pad 1: ROW_38 -> ROW_34
- R34 pad 2: M38 -> M34
- R35 pad 1: ROW_39 -> ROW_35
- R35 pad 2: M39 -> M35
- R36 pad 1: ROW_28 -> ROW_36
- R36 pad 2: M28 -> M36
- R37 pad 1: ROW_29 -> ROW_37
- R37 pad 2: M29 -> M37
- R38 pad 1: ROW_30 -> ROW_38
- R38 pad 2: M30 -> M38
- R39 pad 1: ROW_31 -> ROW_39
- R39 pad 2: M31 -> M39
- R40 pad 1: ROW_32 -> ROW_40
- R40 pad 2: M32 -> M40
- R41 pad 1: ROW_33 -> ROW_41
- R41 pad 2: M33 -> M41
- R42 pad 1: ROW_34 -> ROW_42
- R42 pad 2: M34 -> M42
- R43 pad 1: ROW_35 -> ROW_43
- R43 pad 2: M35 -> M43
- R44 pad 1: ROW_40 -> ROW_44
- R44 pad 2: M40 -> M44
- R45 pad 1: ROW_41 -> ROW_45
- R45 pad 2: M41 -> M45
- R46 pad 1: ROW_42 -> ROW_46
- R46 pad 2: M42 -> M46
- R47 pad 1: ROW_43 -> ROW_47
- R47 pad 2: M43 -> M47
- R48 pad 1: ROW_44 -> ROW_48
- R48 pad 2: M44 -> M48
- R49 pad 1: ROW_45 -> ROW_49
- R49 pad 2: M45 -> M49
- R50 pad 1: ROW_46 -> ROW_50
- R50 pad 2: M46 -> M50
- R51 pad 1: ROW_47 -> ROW_51
- R51 pad 2: M47 -> M51
- R52 pad 1: ROW_48 -> ROW_52
- R52 pad 2: M48 -> M52
- R53 pad 1: ROW_49 -> ROW_53
- R53 pad 2: M49 -> M53
- R54 pad 1: ROW_50 -> ROW_54
- R54 pad 2: M50 -> M54
- R55 pad 1: GNDA -> Net-(U7D--)
- R55 pad 2: Net-(C28-Pad2) -> Net-(R55-Pad2)
- R56 pad 1: GNDA -> Net-(U14D--)
- R56 pad 2: Net-(C56-Pad2) -> Net-(R56-Pad2)
- U1 pad 10: GNDA -> GNDA_ISO
- U1 pad 11: GNDA -> GNDA_ISO
- U1 pad 12: GNDA -> GNDA_ISO
- U1 pad 3: GNDA -> GNDA_ISO
- U1 pad 5: GNDA -> GNDA_ISO
- U10 pad 1: M28 -> M36
- U10 pad 10: GNDA -> GNDA_ISO
- U10 pad 11: GNDA -> GNDA_ISO
- U10 pad 12: GNDA -> GNDA_ISO
- U10 pad 13: ROW_31 -> ROW_39
- U10 pad 14: M31 -> M39
- U10 pad 2: ROW_28 -> ROW_36
- U10 pad 3: GNDA -> GNDA_ISO
- U10 pad 5: GNDA -> GNDA_ISO
- U10 pad 6: ROW_29 -> ROW_37
- U10 pad 7: M29 -> M37
- U10 pad 8: M30 -> M38
- U10 pad 9: ROW_30 -> ROW_38
- U11 pad 1: M32 -> M40
- U11 pad 10: GNDA -> GNDA_ISO
- U11 pad 11: GNDA -> GNDA_ISO
- U11 pad 12: GNDA -> GNDA_ISO
- U11 pad 13: ROW_35 -> ROW_43
- U11 pad 14: M35 -> M43
- U11 pad 2: ROW_32 -> ROW_40
- U11 pad 3: GNDA -> GNDA_ISO
- U11 pad 5: GNDA -> GNDA_ISO
- U11 pad 6: ROW_33 -> ROW_41
- U11 pad 7: M33 -> M41
- U11 pad 8: M34 -> M42
- U11 pad 9: ROW_34 -> ROW_42
- U12 pad 1: M40 -> M44
- U12 pad 10: GNDA -> GNDA_ISO
- U12 pad 11: GNDA -> GNDA_ISO
- U12 pad 12: GNDA -> GNDA_ISO
- U12 pad 13: ROW_43 -> ROW_47
- U12 pad 14: M43 -> M47
- U12 pad 2: ROW_40 -> ROW_44
- U12 pad 3: GNDA -> GNDA_ISO
- U12 pad 5: GNDA -> GNDA_ISO
- U12 pad 6: ROW_41 -> ROW_45
- U12 pad 7: M41 -> M45
- U12 pad 8: M42 -> M46
- U12 pad 9: ROW_42 -> ROW_46
- U13 pad 1: M44 -> M48
- U13 pad 10: GNDA -> GNDA_ISO
- U13 pad 11: GNDA -> GNDA_ISO
- U13 pad 12: GNDA -> GNDA_ISO
- U13 pad 13: ROW_47 -> ROW_51
- U13 pad 14: M47 -> M51
- U13 pad 2: ROW_44 -> ROW_48
- U13 pad 3: GNDA -> GNDA_ISO
- U13 pad 5: GNDA -> GNDA_ISO
- U13 pad 6: ROW_45 -> ROW_49
- U13 pad 7: M45 -> M49
- U13 pad 8: M46 -> M50
- U13 pad 9: ROW_46 -> ROW_50
- U15 pad 3: OUT_0 -> OUT_1
- U16 pad 3: OUT_1 -> OUT_2
- U17 pad 3: OUT_2 -> OUT_3
- U18 pad 3: OUT_3 -> OUT_4
- U19 pad 3: OUT_4 -> OUT_5
- U2 pad 10: GNDA -> GNDA_ISO
- U2 pad 11: GNDA -> GNDA_ISO
- U2 pad 12: GNDA -> GNDA_ISO
- U2 pad 3: GNDA -> GNDA_ISO
- U2 pad 5: GNDA -> GNDA_ISO
- U20 pad 3: OUT_5 -> OUT_6
- U21 pad 3: OUT_6 -> OUT_7
- U22 pad 3: -5VA_ISO -> X0
- U22 pad 6: ENS1_ISO -> ENS1
- U23 pad 3: -5VA_ISO -> X0
- U23 pad 6: ENS2_ISO -> ENS2
- U24 pad 3: -5VA_ISO -> X0
- U24 pad 6: ENS3_ISO -> ENS3
- U25 pad 3: -5VA_ISO -> X0
- U25 pad 6: ENS4_ISO -> ENS4
- U26 pad 3: -5VA_ISO -> X0
- U26 pad 6: ENS5_ISO -> ENS5
- U27 pad 3: -5VA_ISO -> X0
- U27 pad 6: ENS6_ISO -> ENS6
- U28 pad 2: GNDA_ISO -> unconnected-(U28-A6-Pad2)
- U28 pad 3: -5VA_ISO -> X0
- U28 pad 4: GNDA_ISO -> unconnected-(U28-A7-Pad4)
- U28 pad 6: ENS7_ISO -> ENS7
- U3 pad 10: GNDA -> GNDA_ISO
- U3 pad 11: GNDA -> GNDA_ISO
- U3 pad 12: GNDA -> GNDA_ISO
- U3 pad 3: GNDA -> GNDA_ISO
- U3 pad 5: GNDA -> GNDA_ISO
- U4 pad 10: GNDA -> GNDA_ISO
- U4 pad 11: GNDA -> GNDA_ISO
- U4 pad 12: GNDA -> GNDA_ISO
- U4 pad 3: GNDA -> GNDA_ISO
- U4 pad 5: GNDA -> GNDA_ISO
- U6 pad 1: M17 -> M21
- U6 pad 10: GNDA -> GNDA_ISO
- U6 pad 11: GNDA -> GNDA_ISO
- U6 pad 12: GNDA -> GNDA_ISO
- U6 pad 13: ROW_20 -> ROW_24
- U6 pad 14: M20 -> M24
- U6 pad 2: ROW_17 -> ROW_21
- U6 pad 3: GNDA -> GNDA_ISO
- U6 pad 5: GNDA -> GNDA_ISO
- U6 pad 6: ROW_18 -> ROW_22
- U6 pad 7: M18 -> M22
- U6 pad 8: M19 -> M23
- U6 pad 9: ROW_19 -> ROW_23
- U7 pad 1: M21 -> M25
- U7 pad 10: GNDA -> GNDA_ISO
- U7 pad 11: GNDA -> GNDA_ISO
- U7 pad 12: GNDA -> Net-(U7D-+)
- U7 pad 13: ROW_24 -> Net-(U7D--)
- U7 pad 14: M24 -> Net-(R55-Pad2)
- U7 pad 2: ROW_21 -> ROW_25
- U7 pad 3: GNDA -> GNDA_ISO
- U7 pad 5: GNDA -> GNDA_ISO
- U7 pad 6: ROW_22 -> ROW_26
- U7 pad 7: M22 -> M26
- U7 pad 8: M23 -> M27
- U7 pad 9: ROW_23 -> ROW_27
- U8 pad 1: M52 -> M28
- U8 pad 10: GNDA -> GNDA_ISO (x2)
- U8 pad 11: GNDA -> GNDA_ISO (x2)
- U8 pad 12: GNDA -> GNDA_ISO (x2)
- U8 pad 13: GNDA -> ROW_31
- U8 pad 14: Net-(C56-Pad2) -> M31
- U8 pad 2: ROW_52 -> ROW_28
- U8 pad 3: GNDA -> GNDA_ISO (x2)
- U8 pad 5: GNDA -> GNDA_ISO (x2)
- U8 pad 6: ROW_53 -> ROW_29
- U8 pad 7: M53 -> M29
- U8 pad 8: M54 -> M30
- U8 pad 9: ROW_54 -> ROW_30
- U8 pad 1: M48 -> M28
- U8 pad 13: ROW_51 -> ROW_31
- U8 pad 14: M51 -> M31
- U8 pad 2: ROW_48 -> ROW_28
- U8 pad 6: ROW_49 -> ROW_29
- U8 pad 7: M49 -> M29
- U8 pad 8: M50 -> M30
- U8 pad 9: ROW_50 -> ROW_30
- U9 pad 1: M36 -> M32
- U9 pad 10: GNDA -> GNDA_ISO
- U9 pad 11: GNDA -> GNDA_ISO
- U9 pad 12: GNDA -> GNDA_ISO
- U9 pad 13: ROW_39 -> ROW_35
- U9 pad 14: M39 -> M35
- U9 pad 2: ROW_36 -> ROW_32
- U9 pad 3: GNDA -> GNDA_ISO
- U9 pad 5: GNDA -> GNDA_ISO
- U9 pad 6: ROW_37 -> ROW_33
- U9 pad 7: M37 -> M33
- U9 pad 8: M38 -> M34
- U9 pad 9: ROW_38 -> ROW_34
Other:
- board outline added: 229.2 x 50.5 mm
